File: Ece 473 Lab 4 Pre-Amp.brd (EAGLE design)
At the start: 64 x 46 mm, 24 parts, among them J1 2x1, J10 2x1, J11 2x1, J12 2x1, J13 2x1, J2 2x1, J5 2x1, J6 2x1, J8 2x1, J9 2x1

Commit message: Have fun!
Parts:
- removed J11, J12, J13: 2x1, OSU Senior Design:HDRV2W64P254_1X2_467X234X838B
- removed U$1: LMC6032, OSU Senior Design:PDIP-8PIN
- added J3, J4, J7: 2x1, OSU Senior Design:HDRV2W64P254_1X2_467X234X838B
- added U1: LMC6032, OSU Senior Design:PDIP-8PIN
- R3: value 10k -> (none)
- R4: value 10k -> 3k
- R5: value 3k -> 100k
- R6: value (none) -> 100k
- R7, R8: value 100k -> 10k
- moved J8 69.5 mm to (2.54, 43.2), turned to 0 degrees
- moved J6 67.5 mm to (2.54, 2.54), turned to 0 degrees
- moved J9 59.3 mm to (48.3, 2.54), turned to 0 degrees
- moved J10 48.5 mm to (48.3, 20.3), turned to 90 degrees
- moved J5 46.0 mm to (48.3, 25.4), turned to 90 degrees
- moved R5 30.6 mm to (20.3, 40.6)
- moved R8 26.4 mm to (35.6, 7.62)
- moved R3 24.7 mm to (20.3, 15.2)
- moved R4 22.9 mm to (20.3, 10.2)
- moved R7 17.8 mm to (35.6, 22.9)
- moved R6 12.5 mm to (35.6, 27.9)
- moved C3 10.9 mm to (35.6, 33.0)
- moved C4 10.7 mm to (45.7, 10.2), turned to 180 degrees
- moved C1 8.62 mm to (20.3, 35.6)
- moved C2 8.04 mm to (20.3, 20.3)
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Connections:
- net 5V: now also J3.1, R5.2, U1.8; no longer J9.1, R7.2, U$1.8
- net GND: now also J3.2, J4.2, J6.1, J6.2, J7.1, J7.2, J8.2, J9.1, R6.1, U1.4; no longer J10.2, J11.1, J11.2, J12.1, J12.2, J13.1, J13.2, J5.2, R8.1, U$1.4
- net N$1: now also R5.1, R6.2, U1.3, U1.5; no longer R7.1, R8.2, U$1.3, U$1.5
- net N$10: now also R3.2; no longer R6.2
- net N$11: now also R3.1, R4.1, R8.2, U1.6; no longer R4.2, R5.1, R6.1, U$1.6
- net N$12: now also J4.1; no longer J5.1
- net N$13: now also J10.2; no longer J8.2
- net N$5: now also R4.2; no longer R5.2
- net N$6: now also R7.2, U1.2; no longer R3.2, U$1.2
- net N$7: now also J5.2, R7.1, U1.1; no longer J6.2, R3.1, U$1.1
- net N$8: now also J5.1, R8.1, U1.7; no longer J6.1, R4.1, U$1.7
Routing:
- net 5V: track 0.00 -> 61.8 mm
- net N$13: track 0.00 -> 36.7 mm
- net N$1: track 0.00 -> 35.1 mm
- net N$8: track 0.00 -> 25.0 mm
- net N$6: track 0.00 -> 18.2 mm
- net N$12: track 0.00 -> 17.4 mm
- net N$11: track 0.00 -> 15.7 mm
- net N$3: track 0.00 -> 14.3 mm
- net N$5: track 0.00 -> 14.0 mm
- net N$7: track 0.00 -> 13.5 mm
- net N$9: track 0.00 -> 13.2 mm
- net N$4: track 0.00 -> 12.3 mm
- net N$10: track 0.00 -> 12.3 mm
- net N$2: track 0.00 -> 10.3 mm
- added copper zone on layer 1, net GND
Other:
- board size 64 x 46 mm -> 53.3 x 45.7 mm
- board text added: "BUZZ_IN_L"
- board text added: "BUZZ_IN_R"
- board text added: "L_OUT"
- board text added: "RAD_IN_L"
- board text added: "RAD_IN_R"
- board text added: "R_OUT"
- board text added: "VDD"
- board text added: "VOL_IN"
- board text added: "V_OUT"
