File: Ece 473 Lab 4 Pre-Amp.sch (EAGLE design)
At the start: 24 parts, among them J1 2x1, J10 2x1, J11 2x1, J12 2x1, J13 2x1, J2 2x1, J5 2x1, J6 2x1, J8 2x1, J9 2x1

Commit message: Have fun!
Parts:
- removed J11, J13: 2x1, OSU Senior Design:CONNECTOR-2_2X1
- added J3, J4: 2x1, OSU Senior Design:CONNECTOR-2_2X1
- R3: value 10k -> RESISTOR_THROUGH-HOLE; device OSU Senior Design:RESISTOR_10K_THROUGH-HOLE -> OSU Senior Design:RESISTOR_THROUGH-HOLE
- R4: value 10k -> 3k; device OSU Senior Design:RESISTOR_10K_THROUGH-HOLE -> OSU Senior Design:RESISTOR_3K_THROUGH-HOLE
- R5: value 3k -> 100k; device OSU Senior Design:RESISTOR_3K_THROUGH-HOLE -> OSU Senior Design:RESISTOR_100K_THROUGH-HOLE
- R6: value RESISTOR_THROUGH-HOLE -> 100k; device OSU Senior Design:RESISTOR_THROUGH-HOLE -> OSU Senior Design:RESISTOR_100K_THROUGH-HOLE
- R7, R8: value 100k -> 10k; device OSU Senior Design:RESISTOR_100K_THROUGH-HOLE -> OSU Senior Design:RESISTOR_10K_THROUGH-HOLE
- renumbered J12 to J7, U$1 to U1
Connections:
- net 5V: now also J3.1, R5.P$2; no longer J9.1, R7.P$2
- net GND: now also J3.2, J4.2, J6.1, J6.2, J8.2, J9.1, R6.P$1; no longer J10.2, J11.1, J11.2, J13.1, J13.2, J5.2, R8.P$1
- net N$1: now also R5.P$1, R6.P$2; no longer R7.P$1, R8.P$2
- net N$10: now also R3.P$2; no longer R6.P$2
- net N$11: now also R3.P$1, R4.P$1, R8.P$2; no longer R4.P$2, R5.P$1, R6.P$1
- net N$12: now also J4.1; no longer J5.1
- net N$13: now also J10.2; no longer J8.2
- net N$5: now also R4.P$2; no longer R5.P$2
- net N$6: now also R7.P$2; no longer R3.P$2
- net N$7: now also J5.2, R7.P$1; no longer J6.2, R3.P$1
- net N$8: now also J5.1, R8.P$1; no longer J6.1, R4.P$1
Other:
- moved on the sheet: J10, J5, J6, J8, J9, R3, R4, R5, R6, R7, R8
